File: LoRa-TW.kicad_sch (KiCad schematic)
At the start: 38 parts, among them J1 MHF-I/U.FL, U1 SX1262IMLTRT, X1 TCXO, 32MHz, 2.0x1.6mm

Commit message: add shielding can
Parts:
- added C23: 100n, LoRa-TW:C_HF_0402_1005Metric, symbol Device:C_Small
- added J2: Conn_02x06_2.0mm, Connector_PinHeader_2.00mm:PinHeader_2x06_P2.00mm_Vertical, symbol Connector_Generic:Conn_02x06_Odd_Even
- added J3: RFShield_OnePiece, LoRa-TW:ShieldCan, symbol Device:RFShield_OnePiece
- added R10, R4, R5, R6, R7, R8, R9: 33, LoRa-TW:R_HF_0402_1005Metric, symbol Device:R_Small
- L7: footprint LoRa-TW:L_HF_0402_1005Metric -> Inductor_SMD:L_0603_1608Metric
Connections:
- net BUSY: now also R9.2
- net DIO1_INT: now also R10.1
- net GND: now also J2.5 (Pin_5), J2.7 (Pin_7), J3.1 (Shield)
- net MCU_ANT_{SW}: now also J2.11 (Pin_11)
- net SPI_CLK: now also R5.2
- net SPI_MISO: now also R7.2
- net SPI_MOSI: now also R6.2
- net SPI_NSS: now also R4.2
- net VDD: now also C23.2, J2.1 (Pin_1), J2.3 (Pin_3)
- net ~{RESET}: now also C23.1, R8.2
- new net: J2.12 (Pin_12), R9.1
- new net: J2.10 (Pin_10), R8.1
- new net: J2.2 (Pin_2), R4.1
- new net: J2.4 (Pin_4), R5.1
- new net: J2.6 (Pin_6), R6.1
- new net: J2.8 (Pin_8), R7.1
- new net: J2.9 (Pin_9), R10.2
