File: LoRa-TW.kicad_pcb (KiCad board)
At the start: 4 copper layers, 15 x 26.6 mm, 48 parts, among them J1 MHF-I/U.FL, J2 Conn_02x06_2.0mm, J3 RFShield_OnePiece, U1 SX1262IMLTRT, X1 TCXO, 32MHz, 2.0x1.6mm

Commit message: update layout of pcb
Routing:
- net GND: vias 217 -> 219
Other:
- board text added: "BUSY"
- board text added: "CS"
- board text added: "DIO1"
- board text added: "GND"
- board text added: "MISO"
- board text added: "MOSI"
- board text added: "RXEN"
- board text added: "SCLK"
- board text added: "UWINGS KUN-YI LoRaTW_250823"
- board text added: "VCC"
- board text added: "~{RST}"
